File: pcb/ORL.kicad_pcb (KiCad board)
At the start: 2 copper layers, 77.5 x 50.8 mm, 70 parts, among them J1 Conn_01x10_Socket, J10 Conn_01x02_Socket, J11 Conn_01x02_Socket, J12 Conn_01x02_Socket, J13 Conn_01x02_Socket, J14 Conn_01x02_Socket, J15 Conn_01x02_Socket, J16 Conn_01x02_Socket, J17 Conn_01x02_Socket, J18 Conn_01x02_Socket, J19 Conn_01x02_Socket, J2 Conn_01x02_Pin, J20 Conn_01x02_Socket, J21 Conn_01x02_Socket, J22 Conn_01x02_Socket, J23 Conn_01x02_Socket, J24 Conn_01x02_Socket, J25 Conn_01x02_Socket, J26 Conn_01x02_Socket, J27 Conn_01x02_Socket, J28 Conn_01x02_Socket, J29 Conn_01x02_Socket, J3 Conn_01x10_Socket, J30 Conn_01x02_Socket, J31 Conn_01x02_Socket, J32 Conn_01x02_Socket, J33 Conn_01x02_Socket, J4 Conn_02x02_Counter_Clockwise, J5 Conn_02x02_Counter_Clockwise, J6 Conn_02x02_Counter_Clockwise, J7 Conn_02x02_Counter_Clockwise, J8 Conn_02x02_Counter_Clockwise, J9 Conn_02x02_Counter_Clockwise, U1 4071, U2 4071

Commit message: Add reverse polarity protection
Parts:
- added D1: BAT43, Diode_SMD:D_MiniMELF, B.Cu at (157.5, 119.5)
- added D2: BZ5V1, Diode_SMD:D_MiniMELF, B.Cu at (154.9, 119.5)
- added Q1: BUK7880-55A, Package_TO_SOT_SMD:SOT-223-3_TabPin2, B.Cu at (167.0, 119.0)
- added R25: 1k, Resistor_SMD:R_1206_3216Metric, B.Cu at (160.0, 119.8)
- moved FID3 64.3 mm to (102.1, 155.6), turned to 0 degrees
- moved FID1 38.0 mm to (149.9, 84.3)
- moved FID2 35.7 mm to (156.5, 84.3)
- moved R16 7.46 mm to (133.5, 111.8), turned to 180 degrees
- moved R24 3.59 mm to (158.6, 114.3)
Connections:
- J2 pad 2: GND -> Net-(J2-Pin_2)
- J3 pad 1: GND -> Net-(J2-Pin_2)
- J3 pad 10: GND -> Net-(J2-Pin_2)
- J3 pad 2: GND -> Net-(J2-Pin_2)
- J3 pad 3: GND -> Net-(J2-Pin_2)
- J3 pad 4: GND -> Net-(J2-Pin_2)
- J3 pad 5: GND -> Net-(J2-Pin_2)
- J3 pad 6: GND -> Net-(J2-Pin_2)
- J3 pad 7: GND -> Net-(J2-Pin_2)
- J3 pad 8: GND -> Net-(J2-Pin_2)
- J3 pad 9: GND -> Net-(J2-Pin_2)
Routing:
- net Net-(J2-Pin_2): track 0.00 -> 44.0 mm
- net VCC: track 101.6 -> 118.6 mm, vias 3 -> 4
- net Net-(D1-A): track 0.00 -> 8.94 mm
- net Net-(J17-Pin_1): track 19.0 -> 15.4 mm
- net GND: vias 43 -> 49
- added copper zone on B.Cu, net Net-(J2-Pin_2)

Commit message: Optimize fabrication layer
Parts:
- moved FID3 97.1 mm to (168.3, 84.5), turned to 180 degrees
Changed lines of the file:
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@@
   )
   (footprint "Symbol:OSHW-Logo_5.7x6mm_SilkScreen" (layer "B.Cu")
-    (at 102.108 155.575)
+    (at 168.275 84.455 180)
     (descr "Open Source Hardware Logo")
     (tags "Logo OSHW")
@@
         (effects (font (size 0.6 0.6) (thickness 0.12) bold) (justify mirror))
     )
-    (fp_text value "BUK7880-55A" (at 0 -4.5) (layer "B.Fab")
+    (fp_text value "BUK7880-55A" (at 3.15 0 90) (layer "B.Fab")
         (effects (font (size 1 1) (thickness 0.15)) (justify mirror))
     )
@@
         (effects (font (size 0.6 0.6) (thickness 0.12) bold) (justify mirror))
     )
-    (fp_text value "BZ5V1" (at 0 -2 90) (layer "B.Fab")
+    (fp_text value "BZ5V1" (at -4.29 0 90) (layer "B.Fab")
         (effects (font (size 1 1) (thickness 0.15)) (justify mirror))
     )
-    (fp_text user "${REFERENCE}" (at 0 2 90) (layer "B.Fab")
+    (fp_text user "${REFERENCE}" (at 2.695 0 90) (layer "B.Fab")
         (effects (font (size 1 1) (thickness 0.15)) (justify mirror))
     )
@@
         (effects (font (size 0.6 0.6) (thickness 0.12) bold) (justify mirror))
     )
-    (fp_text value "1k" (at 0 -1.82 90) (layer "B.Fab")
+    (fp_text value "1k" (at -2.7325 0 90) (layer "B.Fab")
         (effects (font (size 1 1) (thickness 0.15)) (justify mirror))
     )
@@
         (effects (font (size 0.6 0.6) (thickness 0.12) bold) (justify mirror))
     )
-    (fp_text value "BAT43" (at 0 -2 90) (layer "B.Fab")
+    (fp_text value "BAT43" (at 4.29 0 90) (layer "B.Fab")
         (effects (font (size 1 1) (thickness 0.15)) (justify mirror))
     )
-    (fp_text user "${REFERENCE}" (at 0 2 90) (layer "B.Fab")
+    (fp_text user "${REFERENCE}" (at -2.695 0 90) (layer "B.Fab")
         (effects (font (size 1 1) (thickness 0.15)) (justify mirror))
     )
@@
   (gr_line (start 135.128 126.238) (end 135.128 113.48085)
     (stroke (width 0.15) (type default)) (layer "B.SilkS"))
-  (gr_rect (start 139.1412 126.238) (end 131.064 113.411)
+  (gr_rect (start 131.064 113.411) (end 139.1412 126.238)
     (stroke (width 0.15) (type default)) (fill none) (layer "B.SilkS"))
   (gr_line (start 133.096 126.238) (end 133.096 113.48085)
